Commit message: Everything works fine!

File: four_links/urdf/four_links.urdf (robot description, URDF)
Before this commit: robot four_links, 4 links, 3 joints
Links:
- link linkAB: mass 0.00950214387592875 -> 0.00950214387592874
- link linkBC: mass 0.0178982753669132 -> 0.0180946249077626
Joints:
- joint jointA: origin xyz=-0.126714490675986 0.0295209736544894 -0.0743722309975965 rpy=-1.5707963267949 -1.52106200526056 3.14159265358979 -> xyz=-0.126714490675986 0.0295209736544894 -0.0743722309975965 rpy=1.5707963267949 -1.42221124002695 0
- joint jointB: origin xyz=0.0794339781671298 -0.0353993494464525 -0.02 rpy=0 0 -1.23790614865718 -> xyz=0.074166528159762 0.000154719377460921 -0.00999999999551065 rpy=0 0 -0.982349251785507
- joint jointD: origin xyz=0.0432855093240141 0.0295209736544894 -0.0743722309975965 rpy=1.5707963267949 1.09024680282379 0 -> xyz=0.0432855093240141 0.0295209736544894 -0.0743722309975965 rpy=1.5707963267949 1.18883685572557 0
